File: STM 32 PCB/MCU.kicad_sch (KiCad schematic)
At the start: 40 parts, among them J1 Conn_01x06_MountingPin, J2 Conn_01x03_MountingPin, J3 Conn_01x08_MountingPin, SW1 SW_DIP_x01, U1 STM32F405RGTx, Y1 Crystal

Commit message: 10 dec
Parts:
- added R?: 2k2, symbol Device:R
- C?: renamed from C9; value C -> 100n
- C?: renamed from C2; value 100nF -> 10u
- renumbered C6 to C?, C14 to C?, C11 to C?, C5 to C?, C1 to C?, C16 to C?, C12 to C?, C4 to C?, C17 to C?, C15 to C?, C7 to C?, C13 to C?, C8 to C?, C3 to C?, C10 to C?, D2 to D?, D3 to D?, D1 to D?, D4 to D?, FB1 to FB?, J3 to J?, J2 to J?, J1 to J?, R7 to R?, R6 to R?, R1 to R?, R2 to R?, R11 to R?, R4 to R?, R3 to R?, R9 to R?, R5 to R?, R8 to R?, R10 to R?, SW1 to SW?, TH1 to TH?, U1 to U?, Y1 to Y?
Connections:
- net GND: now also R?.1; no longer SW?.1
- net SCK_ADC_EXT: now reaches J?.4 (Pin_4)
- net SCK_ADC_EXT: now also U?.21 (PA5)
- net TX_SDA_NSS: now reaches J?.5 (Pin_5)
- net TX_SDA_NSS: now also U?.20 (PA4), U?.30 (PB11)
- net RX_SCL_MOS: now reaches J?.6 (Pin_6)
- net MISO_ADC_EXT2: now reaches J?.7 (Pin_7)
- net MISO_ADC_EXT2: now also U?.22 (PA6)
- net AN_J: now reaches C?.1, R?.1, R?.2
- net ADC_TEMP: now reaches R?.2, TH?.2
- net ADC_TEMP: now also U?.17 (PA3)
- net AN_IN: now reaches U?.10 (PC2)
- net SENS3: now reaches U?.14 (PA0)
- net SENS2: now reaches U?.15 (PA1)
- net SENS1: now reaches U?.16 (PA2)
- net RX_SCL_MOSI: now reaches U?.23 (PA7)
- net RX_SCL_MOSI: now also U?.29 (PB10)
- net BR_S02: now reaches U?.26 (PB0)
- net BR_S01: now reaches U?.27 (PB1)
- net DC_CAL: now reaches U?.33 (PB12)
- net L3: now reaches U?.34 (PB13)
- net L2: now reaches U?.35 (PB14)
- net L1: now reaches U?.36 (PB15)
- net LED_SDA_NSS: now reaches U?.37 (PC6)
- net LED_SCL_MOSI: now reaches U?.38 (PC7)
- net H3: now reaches U?.41 (PA8)
- net H2: now reaches U?.42 (PA9)
- net H1: now reaches U?.43 (PA10)
- net USB_DM: now reaches U?.44 (PA11)
- net USB_DP: now reaches U?.45 (PA12)
- net SWDIO: now reaches U?.46 (PA13)
- net SWDIO: now also J?.4 (Pin_4)
- net SWCLK: now reaches U?.49 (PA14)
- net SWCLK: now also J?.2 (Pin_2)
- net EN_GATE: now reaches U?.51 (PC10)
- net HALL_3: now reaches U?.52 (PC11)
- net FAULT: now reaches U?.53 (PC12)
- net SERVO: now reaches U?.57 (PB5)
- net HALL_1: now reaches U?.58 (PB6)
- net HALL_2: now reaches U?.59 (PB7)
- net CAN_RX: now reaches U?.61 (PB8)
- net CAN_TX: now reaches U?.62 (PB9)
- net Temp_Motor: now reaches U?.8 (PC0)
- net NRST: now reaches J?.5 (Pin_5)
- new net: R?.2, SW?.1
- no-connect marks 0 -> 11
Other:
- note removed: "ADC_TEMP"
- note removed: "AN_IN"
- note removed: "AN_JN"
- note removed: "BR_S01"
- note removed: "BR_S02"
- note removed: "CAN_RX"
- note removed: "CAN_TX"
- note removed: "DC_CAL"
- note removed: "EN_GATE"
- note removed: "FAULT"
- note removed: "H1"
- note removed: "H2"
- note removed: "H3"
- note removed: "HALL_1"
- note removed: "HALL_2"
- note removed: "HALL_3"
- note removed: "L1"
- note removed: "L2"
- note removed: "L3"
- note removed: "LED_SCL_MOSI"
- note removed: "LED_SDA_NSS"
- note removed: "MISO_ADC_EXT2"
- note removed: "RX_SCL_MOSI"
- note removed: "SCK_ADC_EXT"
- note removed: "SENS1"
- note removed: "SENS2"
- note removed: "SENS3"
- note removed: "SWCLK"
- note removed: "SWDIO"
- note removed: "TX_SDA_NSS"
- note removed: "Temp_Motor"
- note removed: "USB_DM"
- note removed: "USB_DP"
- moved on the sheet: C?
