File: STM 32 PCB/MOSFET Driver.kicad_sch (KiCad schematic)
At the start: 18 parts, among them U2 DRV8302_DCA_56

Commit message: 10 dec
Parts:
- removed R12: R, symbol Device:R
- added C? (x6): 1u, symbol Device:C
- added C? (x3): 220n, symbol Device:C
- added C?: 100n, symbol Device:C
- added C? (x3): 10u, symbol Device:C
- added C?: 0.015u, symbol Device:C
- added D?: PMEG6020AELR, Diode_SMD:Nexperia_CFP3_SOD-123W, symbol Diode:PMEG6020AELR
- added D?: BAT60A, Diode_SMD:D_SOD-323, symbol Diode:BAT60A
- added L?: 22u, symbol Device:L
- added R? (x3): 39K, symbol Device:R
- added R? (x3): 2K2, symbol Device:R
- added R?: 1M, symbol Device:R
- added R?: 18K, symbol Device:R
- added R?: 3K3, symbol Device:R
- renumbered C25 to C?, C24 to C?, C18 to C?, C27 to C?, C22 to C?, C23 to C?, C28 to C?, C20 to C?, C19 to C?, C26 to C?, C21 to C?, R15 to R?, R13 to R?, R14 to R?, R17 to R?, R16 to R?, U2 to U?
Connections:
- net +3V3: now also U?.24 (REF)
- net +5V: now also D?.1 (K)
- net BR_SO1: now also U?.25 (SO1)
- net BR_SO2: now also U?.26 (SO2)
- net DVDD: now also U?.23 (DVDD)
- net EN_GATE: now also U?.16 (EN_GATE)
- net GND: now also U?.57 (EPAD), C?.1, C?.1, C?.1, C?.1, C?.2, C?.2, C?.2, C?.2, C?.2, C?.2, D?.2 (A), R?.2, R?.2, R?.2, R?.2, R?.2
- net H1: now also U?.17 (INH_A)
- net H2: now also U?.19 (INH_B)
- net H3: now also U?.21 (INH_C)
- net L1: now also U?.18 (INL_A)
- net L2: now also U?.20 (INL_B)
- net L3: now also U?.22 (INL_C)
- net RT_CLK: now reaches R?.2, U?.1 (RT_CLK)
- net OC_ADJ: now reaches C?.1, C?.1, U?.11 (OC_ADJ)
- net GVDD: now reaches C?.1, C?.1, U?.13 (GVDD)
- net COMP: now reaches C?.2, R?.2, U?.2 (COMP)
- net +VDC: now reaches C?.1, C?.1, C?.1, U?.29 (PVDD1)
- net +VDC: now also U?.53 (PVDD2), U?.54 (PVDD2), C?.1, C?.1, C?.1, C?.1, C?.1, C?.1
- net VSENSE: now reaches R?.1, R?.2, U?.3 (VSENSE)
- net VSENSE: now also R?.1
- net S2_P: now reaches U?.30 (SP2)
- net S2_N: now reaches U?.31 (SN2)
- net S1_P: now reaches U?.32 (SP1)
- net S1_N: now reaches U?.33 (SN1)
- net H3_LOW: now reaches U?.34 (SL_C)
- net M_L3: now reaches U?.35 (GL_C)
- net H3_VS: now reaches U?.36 (SH_C)
- net H3_VS: now also C?.1, R?.1
- net M_H3: now reaches U?.37 (GH_C)
- net BST_C: now reaches U?.38 (BST_C)
- net BST_C: now also C?.2
- net H2_LOW: now reaches U?.39 (SL_B)
- net M_L2: now reaches U?.40 (GL_B)
- net H2_VS: now reaches U?.41 (SH_B)
- net H2_VS: now also C?.1, R?.1
- net M_H2: now reaches U?.42 (GH_B)
- net BST_B: now reaches U?.43 (BST_B)
- net BST_B: now also C?.2
- net H1_LOW: now reaches U?.44 (SL_A)
- net M_L1: now reaches U?.45 (GL_A)
- net H1_VS: now reaches U?.46 (SH_A)
- net H1_VS: now also C?.1, R?.1
- net M_H1: now reaches U?.47 (GH_A)
- net BST_A: now reaches U?.48 (BST_A)
- net BST_A: now also C?.2
- net BIAS: now reaches U?.49 (BIAS)
- net BIAS: now also R?.1
- net PH: now reaches U?.50 (PH)
- net PH: now also U?.51 (PH), C?.2, D?.1 (K), L?.1
- net BST_BK: now reaches U?.52 (BST_BK)
- net BST_BK: now also C?.1
- net at U?.56 (SS_TR): now also C?.2
- net DTC: now reaches R?.2, U?.7 (DTC)
- net M_OC: now reaches U?.9 (M_OC)
- new net +5V_DRV: C?.2, C?.2, C?.2, D?.2 (A), L?.2
- new net SENS1: R?.1, R?.2
- new net SENS2: R?.1, R?.2
- new net SENS3: R?.1, R?.2
- no-connect marks 0 -> 3
Other:
- note added: "1u DECOUPLING PLACE AS CLOSE AS POSSIBLE TO IC"
- note added: "BOOTSTRAP CAPs"
- note added: "Hx_VS"
- note added: "KEEP AWAY FROM NOISE TRACKS AND COMPONENTS"
- note added: "MCU SENSING FEEDBACK FOR EACH PHASE"
- note added: "MOSFET DRIVER"
- note added: "OUT PUT PORTS"
- note added: "PHASE_1"
- note added: "PHASE_2"
- note added: "PHASE_3"
- note added: "SENSE 1 - PHASE 3"
- note added: "SENSE 2 - PHASE 2"
- note added: "keeping as close as possible to ic and to driver input loop"
- note removed: "+3V3"
- note removed: "BR_SO1"
- note removed: "BR_SO2"
- note removed: "EN_GATE"
- note removed: "H1"
- note removed: "H2"
- note removed: "H3"
- note removed: "L1"
- note removed: "L2"
- note removed: "L3"
