File: STM 32 PCB/CAN.kicad_sch (KiCad schematic)
At the start: 0 parts

Commit message: 11 Dec
Parts:
- added C5: C, symbol Device:C
- added R10, R11, R8, R9: R, symbol Device:R
- added U1: SN65HVD230, Package_SO:SOIC-8_3.9x4.9mm_P1.27mm, symbol Interface_CAN_LIN:SN65HVD230
Connections:
- new net: C5.2, R9.1
- new net GND: C5.1, R9.2
Other:
- note added: "CAN_H AND CAN_L TO BE ROUTED AS DIFFERENTIAL PAIR"

Commit message: 1
Parts:
- added C6: 60p, symbol Device:C
- added D3: ESDCAN24-2BLY, SOT95P255X125-3N, symbol ESDCAN24-2BLY:ESDCAN24-2BLY
- added L1: 744227S, WE-SL274, symbol 744227S:744227S
- C5: value C -> 60p
- R10, R11: value R -> 10R
- R9: value R -> 120R
Connections:
- net GND: now also C6.2, D3.3 (I/O_3); no longer R9.2
- net at C5.2, R9.1: now also R10.1, D3.1 (I/O_1)
- net at R10.2: now also L1.1
- net at R11.1: now also R9.2, C6.1, D3.2 (I/O_2)
- net at R11.2: now also L1.2 (3)
- net at U1.6 (CANL): now also L1.3 (4)
- net at U1.7 (CANH): now also L1.4 (2)
- no-connect marks 0 -> 1
Other:
- note added: "[07] CAN"
- moved on the sheet: U1
