File: esp_Extension/esp_Extension.kicad_sch (KiCad schematic)
At the start: 3 parts, among them P1 Connector_Generic:Conn_01x08, P2 Connector_Generic:Conn_01x08, U1 WeMos_D1_mini

Commit message: 1
Parts:
- removed P1, P2: Connector_Generic:Conn_01x08, D1_mini:D1_mini_Pin_Header, symbol Connector_Generic:Conn_01x08
- added D1: LED, LED_THT:LED_D5.0mm, symbol PCM_SL_Devices:LED
- added J1: Conn_01x08_Pin L, Connector_PinHeader_2.54mm:PinHeader_1x08_P2.54mm_Vertical, symbol Connector:Conn_01x08_Pin
- added J2: Conn_01x05_Pin G, Connector_PinHeader_2.54mm:PinHeader_1x05_P2.54mm_Vertical, symbol Connector:Conn_01x05_Pin
- added J3: Conn_01x08_Pin L, TerminalBlock_RND:TerminalBlock_RND_205-00018_1x08_P5.00mm_Horizontal, symbol Connector:Conn_01x08_Pin
- added J4: Conn_01x05_Pin 5v, Connector_PinHeader_2.54mm:PinHeader_1x05_P2.54mm_Vertical, symbol Connector:Conn_01x05_Pin
- added J5: Conn_01x08_Pin R, TerminalBlock_RND:TerminalBlock_RND_205-00018_1x08_P5.00mm_Horizontal, symbol Connector:Conn_01x08_Pin
- added J6: Conn_01x05_Pin3.3v, Connector_PinHeader_2.54mm:PinHeader_1x05_P2.54mm_Vertical, symbol Connector:Conn_01x05_Pin
- added J7: Conn_01x08_Pin R, Connector_PinHeader_2.54mm:PinHeader_1x08_P2.54mm_Vertical, symbol Connector:Conn_01x08_Pin
- added R1: R, Resistor_THT:R_Axial_DIN0207_L6.3mm_D2.5mm_P7.62mm_Horizontal, symbol PCM_Elektuur:R
- added SW1: SW_Push, Button_Switch_THT:SW_PUSH_6mm_H5mm, symbol Switch:SW_Push
- added U2, U3, U4: WeMos_D1_mini, Module:WEMOS_D1_mini_light, symbol MCU_Module:WeMos_D1_mini
Connections:
- net GND: now also U1.10 (GND), D1.1, J2.1 (Pin_1), J2.2 (Pin_2), J2.3 (Pin_3), J2.4 (Pin_4), J2.5 (Pin_5), J5.7 (Pin_7), J7.7 (Pin_7), SW1.1
- net at U1.1 (~{RST}): now also J1.1 (Pin_1), J3.1 (Pin_1), SW1.2
- net at U1.11 (D4): now also J5.6 (Pin_6), J7.6 (Pin_6), U2.11 (D4), U3.11 (D4), U4.11 (D4)
- net at U1.12 (D3): now also J5.5 (Pin_5), J7.5 (Pin_5), U2.12 (D3), U3.12 (D3), U4.12 (D3)
- net at U1.13 (SDA/D2): now also J5.4 (Pin_4), J7.4 (Pin_4), U2.13 (SDA/D2), U3.13 (SDA/D2), U4.13 (SDA/D2)
- net at U1.14 (SCL/D1): now also J5.3 (Pin_3), J7.3 (Pin_3), U2.14 (SCL/D1), U3.14 (SCL/D1), U4.14 (SCL/D1)
- net at U1.15 (RX): now also J5.2 (Pin_2), J7.2 (Pin_2)
- net at U1.16 (TX): now also J5.1 (Pin_1), J7.1 (Pin_1)
- net at U1.2 (A0): now also J1.2 (Pin_2), J3.2 (Pin_2), U2.2 (A0), U3.2 (A0), U4.2 (A0)
- net at U1.3 (D0): now also J1.3 (Pin_3), J3.3 (Pin_3), U2.3 (D0), U3.3 (D0), U4.3 (D0)
- net at U1.4 (SCK/D5): now also J1.4 (Pin_4), J3.4 (Pin_4), U2.4 (SCK/D5), U3.4 (SCK/D5), U4.4 (SCK/D5)
- net at U1.5 (MISO/D6): now also J1.5 (Pin_5), J3.5 (Pin_5), U2.5 (MISO/D6), U2.6 (MOSI/D7), U3.5 (MISO/D6), U3.6 (MOSI/D7), U4.5 (MISO/D6), U4.6 (MOSI/D7)
- net at U1.6 (MOSI/D7): now also J1.6 (Pin_6), J3.6 (Pin_6)
- net at U1.7 (CS/D8): now also J1.7 (Pin_7), J3.7 (Pin_7), U2.7 (CS/D8), U3.7 (CS/D8), U4.7 (CS/D8)
- net at U1.8 (3V3): now also J1.8 (Pin_8), J3.8 (Pin_8), J6.1 (Pin_1), J6.2 (Pin_2), J6.3 (Pin_3), J6.4 (Pin_4), J6.5 (Pin_5)
- net at U1.9 (5V): now also J4.1 (Pin_1), J4.2 (Pin_2), J4.3 (Pin_3), J4.4 (Pin_4), J4.5 (Pin_5), J5.8 (Pin_8), J7.8 (Pin_8), R1.1 (+)
- new net: U2.1 (~{RST}), U3.1 (~{RST}), U4.1 (~{RST})
- new net: U2.10 (GND), U3.10 (GND), U4.10 (GND)
- new net: U2.15 (RX), U3.15 (RX), U4.15 (RX)
- new net: U2.16 (TX), U3.16 (TX), U4.16 (TX)
- new net: U2.8 (3V3), U3.8 (3V3), U4.8 (3V3)
- new net: U2.9 (5V), U3.9 (5V), U4.9 (5V)
- new net: D1.2, R1.2 (-)
Other:
- note added: "3.3 D8 D7 D6 D5 D0 A0 RS"
- note added: "5V G D4 D3 D2 D1 RX TX"
- note removed: "D1 Mini Shield"
- note removed: "GPIO0"
- note removed: "GPIO12"
- note removed: "GPIO13"
- note removed: "GPIO14"
- note removed: "GPIO15"
- note removed: "GPIO16"
- note removed: "GPIO2"
- note removed: "GPIO4"
- note removed: "GPIO5"
- moved on the sheet: U1
