File: esp_Extension/esp_Extension.kicad_pcb (KiCad board)
At the start: 2 copper layers, 99 x 99.5 mm, 14 parts, among them J1 Conn_01x08_Pin L, J2 Conn_01x05_Pin G, J3 Conn_01x08_Pin L, J4 Conn_01x05_Pin 5v, J5 Conn_01x08_Pin R, J6 Conn_01x05_Pin3.3v, J7 Conn_01x08_Pin R, SW1 SW_Push, U1 WeMos_D1_mini, U2 WeMos_D1_mini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

Commit message: 21
Parts:
- moved J1 0.29 mm to (45.7, 69.5)
Routing:
- net Net-(J4-Pin_1): track 106.3 -> 110.0 mm
- net Net-(J5-Pin_4): track 144.1 -> 146.1 mm
- net Net-(J1-Pin_2): track 172.1 -> 174.0 mm
- net Net-(J1-Pin_5): track 180.0 -> 181.6 mm
- net Net-(J1-Pin_7): track 172.1 -> 173.7 mm
- net Net-(J1-Pin_3): track 169.6 -> 170.9 mm
- net Net-(J1-Pin_8): track 130.3 -> 131.6 mm
- net Net-(J1-Pin_6): track 116.1 -> 117.4 mm
- net Net-(J1-Pin_4): track 171.2 -> 172.2 mm
- net Net-(J5-Pin_3): track 144.5 -> 145.5 mm
- net Net-(J5-Pin_6): track 142.0 -> 143.0 mm
Other:
- outline, holes or cut-outs redrawn
